File: PCB/ADC_DAC_Converter/DAC_Converter - KiCAD/ADC_DAC_Converter.kicad_sch (KiCad schematic)
At the start: 8 parts, among them SW1 SW_SPST, SW2 SW_SPST, SW3 SW_SPST, U1 OP1177ARM

Commit message: PCB Design Completed
Parts:
- added C1: 200n, Capacitor_THT:C_Axial_L3.8mm_D2.6mm_P7.50mm_Horizontal, symbol Device:C
- added R5: 1k, Resistor_THT:R_Axial_DIN0207_L6.3mm_D2.5mm_P15.24mm_Horizontal, symbol Device:R_US
- SW1, SW2, SW3: footprint (none) -> Button_Switch_THT:SW_DIP_SPSTx01_Slide_6.7x4.1mm_W7.62mm_P2.54mm_LowProfile
Connections:
- net GND: now also C1.2
- net OUT: now also R5.1
- new net Analog_Out: C1.1, R5.2
Other:
- note added: "First-order Lowpass Filter"
- company: (none) -> Elektronica
- title: (none) -> DAC Converter
